File: First Round Clock/First Round Clock.kicad_sch (KiCad schematic)
At the start: 43 parts, among them J1 Power_inlet_vertical, J2 Conn_01x06, J3 Conn_02x03_Odd_Even, Q1 NPN_2N3904_SOT23, SW1 Omron_B3F_SPST, SW2 Omron_B3F_SPST, SW3 Omron_B3F_SPST, SW4 Omron_B3F_SPST, SW5 Omron_B3F_SPST, U1 L7805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

Commit message: Final clock
Final gerber out for clock
Parts:
- added TP1, TP10, TP11, TP12, TP13, TP14, TP15, TP16, TP17, TP2, TP3, TP4, TP5, TP6, TP7, TP8, TP9: TestPoint, footprints:TestPoint_THTPad_D2.0mm_Drill1.0mm, symbol HPS:TestPoint
Connections:
- net LED_SCK: now also TP7.1
- net LIGHT_SENSOR: now also TP10.1
- net MISO: now also TP12.1
- net MOSI: now also TP14.1
- net RESET: now also TP8.1
- net SCL: now also TP6.1
- net SDA: now also TP5.1
- net VCC: now also TP1.1, TP13.1
- net at U3.1 (X1), Y2.2: now also TP16.1
- net at U3.2 (X2), Y2.1: now also TP17.1
- net at BT1.1 (+), U3.3 (VBAT): now also TP15.1
- net at C3.1, J1.1 (POLE), U1.1 (IN): now also TP3.1
- net at C2.2, U2.9 (XTAL1/PB6), Y1.2: now also TP2.1
- net at Q1.1 (B), R8.2: now also TP9.1
- net at J2.4 (Pin_4), R2.2: now also TP4.1
- net at DS1.3 (VO), RV1.2: now also TP11.1

Commit message: final fix for clock
Final clock used and fixed
Parts:
- removed TP13, TP17, TP4: TestPoint, footprints:TestPoint_THTPad_D2.0mm_Drill1.0mm, symbol HPS:TestPoint
- added C7: C_0805_1uf, footprints:C_0805_2012Metric, symbol HPS:C_0805_1uf
Connections:
- net GND: now also C7.2
- net VCC: now also C3.1
- net at J1.1 (POLE), TP3.1, U1.1 (IN): now also C7.1; no longer C3.1
